File: kicad/mikrokontrolleri/mikrokontrolleri.sch (KiCad schematic (older format))
At the start: 16 parts, among them SW1 SW_Push, SW2 SW_Push, SW3 SW_Push, U1 ATmega328P, U1 MCP3202, Y1 16MHz

Commit message: Muutokset kaavioihin.
Parts:
- added BZ1: Buzzer, symbol Device:Buzzer
- added C7, C8: 22u, symbol Device:C
- added C9: 1u, symbol Device:C
- added R2: 100, symbol Device:R
Connections:
- net GND: now also U?.4 (VSS), BZ1.2 (+), C7.2, C8.1
- net SCL: now also U?.6 (SCL)
- net SDA: now also U?.5 (SDA)
- net VCC: now also U?.8 (VCC), C7.1
- net BZ: now reaches U1.5 (PD3)
- net BZ: now also R2.2
- net at U?.1 (VCAP): now also C8.2
- new net: BZ1.1 (-), C9.2
- new net: C9.1, R2.1
- no-connect marks 9 -> 11
Changed lines of the file:
@@
 P 4250 4550
 F 0 "#PWR?" H 4250 4300 50  0001 C CNN
-F 1 "GND" H 4255 4377 50  0000 C CNN
+F 1 "GND" H 4250 4400 50  0000 C CNN
 F 2 "" H 4250 4550 50  0001 C CNN
 F 3 "" H 4250 4550 50  0001 C CNN
@@
 Wire Wire Line
 	5300 2500 5550 2500
-Wire Bus Line
-	3600 2600 5200 2600
 $Comp
 L Device:C C3
@@
 MOSI
 NoConn ~ 3350 3800
-NoConn ~ 3350 3900
 NoConn ~ 3350 4100
 NoConn ~ 3350 4200
@@
 L Memory_NVRAM:47C16 U?
 U 1 1 61B8864D
-P 4400 5300
-F 0 "U?" H 4400 4811 50  0001 C CNN
-F 1 "47C16" H 4400 4811 50  0000 C CNN
-F 2 "" H 4400 4850 50  0001 C CNN
-F 3 "http://ww1.microchip.com/downloads/en/DeviceDoc/20005371C.pdf" H 4650 5650 50  0001 C CNN
-	1    4400 5300
-	1    0    0    -1
-$EndComp
-Entry Wire Line
-	3600 5350 3700 5250
-Entry Wire Line
-	3600 5450 3700 5350
-Text Label 3700 5250 0    50   ~ 0
+P 4250 5500
+F 0 "U?" H 4250 5011 50  0001 C CNN
+F 1 "47C16" H 3950 5100 50  0000 C CNN
+F 2 "" H 4250 5050 50  0001 C CNN
+F 3 "http://ww1.microchip.com/downloads/en/DeviceDoc/20005371C.pdf" H 4500 5850 50  0001 C CNN
+	1    4250 5500
+	1    0    0    -1
+$EndComp
+Entry Wire Line
+	3600 5500 3700 5400
+Entry Wire Line
+	3600 5600 3700 5500
+Text Label 3700 5400 0    50   ~ 0
 SCL
-Text Label 3700 5350 0    50   ~ 0
+Text Label 3700 5500 0    50   ~ 0
 SDA
-Wire Wire Line
-	3700 5250 3850 5250
-Wire Wire Line
-	3700 5350 3850 5350
 Entry Wire Line
 	3600 3400 3500 3300
@@
 Wire Wire Line
 	3500 3200 3350 3200
+Wire Wire Line
+	3700 5500 3850 5500
+Wire Wire Line
+	3700 5400 3850 5400
+NoConn ~ 4650 5500
+NoConn ~ 4650 5600
+NoConn ~ 3850 5700
+$Comp
+L power:GND #PWR?
+U 1 1 61E9BA5B
+P 4250 5950
+F 0 "#PWR?" H 4250 5700 50  0001 C CNN
+F 1 "GND" H 4255 5777 50  0000 C CNN
+F 2 "" H 4250 5950 50  0001 C CNN
+F 3 "" H 4250 5950 50  0001 C CNN
+	1    4250 5950
+	1    0    0    -1
+$EndComp
+Wire Wire Line
+	4250 5900 4250 5950
+$Comp
+L Device:C C7
+U 1 1 61EA8051
+P 4050 5100
+F 0 "C7" V 3798 5100 50  0000 C CNN
+F 1 "22u" V 3889 5100 50  0000 C CNN
+F 2 "" H 4088 4950 50  0001 C CNN
+F 3 "~" H 4050 5100 50  0001 C CNN
+	1    4050 5100
+	0    1    1    0
+$EndComp
+Wire Wire Line
+	3900 5100 3850 5100
+Wire Wire Line
+	3850 5100 3850 5150
+$Comp
+L power:VCC #PWR?
+U 1 1 61EAC74A
+P 4250 5000
+F 0 "#PWR?" H 4250 4850 50  0001 C CNN
+F 1 "VCC" H 4250 5150 50  0000 C CNN
+F 2 "" H 4250 5000 50  0001 C CNN
+F 3 "" H 4250 5000 50  0001 C CNN
+	1    4250 5000
+	1    0    0    -1
+$EndComp
+$Comp
+L power:GND #PWR?
+U 1 1 61EC2088
+P 3850 5150
+F 0 "#PWR?" H 3850 4900 50  0001 C CNN
+F 1 "GND" H 3750 5150 50  0000 C CNN
+F 2 "" H 3850 5150 50  0001 C CNN
+F 3 "" H 3850 5150 50  0001 C CNN
+	1    3850 5150
+	1    0    0    -1
+$EndComp
+Wire Wire Line
+	4250 5000 4250 5100
+Wire Wire Line
+	4200 5100 4250 5100
+Connection ~ 4250 5100
+Wire Wire Line
+	4250 5100 4250 5200
+$Comp
+L Device:C C8
+U 1 1 61EDFE45
+P 4550 5100
+F 0 "C8" V 4298 5100 50  0000 C CNN
+F 1 "22u" V 4389 5100 50  0000 C CNN
+F 2 "" H 4588 4950 50  0001 C CNN
+F 3 "~" H 4550 5100 50  0001 C CNN
+	1    4550 5100
+	0    1    1    0
+$EndComp
+$Comp
+L power:GND #PWR?
+U 1 1 61EE079A
+P 4750 5150
+F 0 "#PWR?" H 4750 4900 50  0001 C CNN
+F 1 "GND" H 4900 5150 50  0000 C CNN
+F 2 "" H 4750 5150 50  0001 C CNN
+F 3 "" H 4750 5150 50  0001 C CNN
+	1    4750 5150
+	1    0    0    -1
+$EndComp
+Wire Wire Line
+	4750 5150 4750 5100
+Wire Wire Line
+	4750 5100 4700 5100
+Wire Wire Line
+	4400 5100 4350 5100
+Wire Wire Line
+	4350 5100 4350 5200
+Entry Wire Line
+	3500 3900 3600 4000
+Wire Wire Line
+	3500 3900 3350 3900
+Text Label 3400 3900 0    50   ~ 0
+BZ
+$Comp
+L Device:Buzzer BZ1
+U 1 1 61F299A8
+P 5100 2150
+F 0 "BZ1" H 5252 2179 50  0000 L CNN
+F 1 "Buzzer" H 5252 2088 50  0000 L CNN
+F 2 "" V 5075 2250 50  0001 C CNN
+F 3 "~" V 5075 2250 50  0001 C CNN
+	1    5100 2150
+	1    0    0    -1
+$EndComp
+$Comp
+L Device:R R2
+U 1 1 61F2AED5
+P 4600 2250
+F 0 "R2" H 4670 2296 50  0000 L CNN
+F 1 "100" H 4670 2205 50  0000 L CNN
+F 2 "" V 4530 2250 50  0001 C CNN
+F 3 "~" H 4600 2250 50  0001 C CNN
+	1    4600 2250
+	1    0    0    -1
+$EndComp
+$Comp
+L Device:C C9
+U 1 1 61F2B5C8
+P 4800 2050
+F 0 "C9" V 5052 2050 50  0000 C CNN
+F 1 "1u" V 4961 2050 50  0000 C CNN
+F 2 "" H 4838 1900 50  0001 C CNN
+F 3 "~" H 4800 2050 50  0001 C CNN
+	1    4800 2050
+	0    -1   -1   0
+$EndComp
+Entry Wire Line
+	4500 2600 4600 2500
+Wire Wire Line
+	4600 2500 4600 2400
+Text Label 4600 2500 0    50   ~ 0
+BZ
+$Comp
+L power:GND #PWR?
+U 1 1 61F72545
+P 4950 2300
+F 0 "#PWR?" H 4950 2050 50  0001 C CNN
+F 1 "GND" H 4955 2127 50  0000 C CNN
+F 2 "" H 4950 2300 50  0001 C CNN
+F 3 "" H 4950 2300 50  0001 C CNN
+	1    4950 2300
+	1    0    0    -1
+$EndComp
+Wire Wire Line
+	4950 2300 4950 2250
+Wire Wire Line
+	4950 2250 5000 2250
+Wire Wire Line
+	5000 2050 4950 2050
+Wire Wire Line
+	4600 2100 4600 2050
+Wire Wire Line
+	4600 2050 4650 2050
+Wire Bus Line
+	3600 2600 5200 2600
 Wire Bus Line
 	5200 2600 5200 3500
