File: kicad/vahvistin/vahvistin.sch (KiCad schematic (older format))
At the start: 17 parts, among them U1 LM324, U2 LM324, U3 LM324, U4 LM324

Commit message: Muutokset kaavioihin.
Parts:
- added R5, R6: 5.6k, symbol Device:R
- added R7: 680, symbol Device:R
- R10: renamed from R7; value 6.8k -> 33k
- R11: renamed from R8; value 8.2k -> 33k
- R8: renamed from R5; value 120 -> 8.2k
- R9: renamed from R6; value 100 -> 8.2k
- renumbered R9 to R12, R10 to R13
Connections:
- net at R8.2, U1.1: now also R5.2, R7.2; no longer U1.2 (-)
- net at R9.1, U2.1: now also R6.2, R7.1; no longer U2.2 (-)
- new net: R5.1, U1.2 (-)
- new net: R6.1, U2.2 (-)
Other:
- note added: "Instrumentointivahvistin"
- note removed: "Differentiaalivahvistin"
- note removed: "Puskurointi\n´"
- moved on the sheet: R10, R11, R8, R9
